Commit message: [tb3_sim_waffle] TB3 waffle simulator added

File: tb3_sim/urdf/turtlebot3_waffle.urdf (robot description, URDF)
Before this commit: robot turtlebot3_waffle, 8 links, 7 joints
Links:
- added link camera_depth_frame
- added link camera_depth_optical_frame
- added link camera_link; collision box size=0.012 0.132 0.020; visual mesh filename=package://turtlebot3_description/meshes/sensors/r200.dae
- added link camera_rgb_frame
- added link camera_rgb_optical_frame
Joints:
- added joint camera_depth_joint: type fixed, parent camera_link, child camera_depth_frame, origin xyz=0.005 0.028 0.013 rpy=-1.57 0 -1.57
- added joint camera_depth_optical_joint: type fixed, parent camera_depth_frame, child camera_depth_optical_frame, origin xyz=0 0 0 rpy=0 0 0
- added joint camera_joint: type fixed, parent base_link, child camera_link, origin xyz=0.064 -0.065 0.094 rpy=0 0 0
- added joint camera_rgb_joint: type fixed, parent camera_link, child camera_rgb_frame, origin xyz=0.005 0.018 0.013 rpy=0 0 0
- added joint camera_rgb_optical_joint: type fixed, parent camera_rgb_frame, child camera_rgb_optical_frame, origin xyz=0 0 0 rpy=-1.57 0 -1.57
